Commit message: More cleaning

File: finger.urdf (robot description, URDF)
Before this commit: robot finger, 22 links, 21 joints
Links:
- added link act0Seg11, mass 0.35; collision box size=0.2 0.2 0.2; visual box size=0.2 0.2 0.2
- added link act0Seg11helper_shape, mass 0.00035; collision cylinder length=0.2 radius=0.1; visual cylinder length=0.2 radius=0.1
- added link act0Seg12, mass 0.35; collision box size=0.2 0.2 0.2; visual box size=0.2 0.2 0.2
- added link act0Seg12helper_shape, mass 0.00035; collision cylinder length=0.2 radius=0.1; visual cylinder length=0.2 radius=0.1
- added link act0Seg13, mass 0.35; collision box size=0.2 0.2 0.2; visual box size=0.2 0.2 0.2
- added link act0Seg13helper_shape, mass 0.00035; collision cylinder length=0.2 radius=0.1; visual cylinder length=0.2 radius=0.1
- added link act0Seg14, mass 0.35; collision box size=0.2 0.2 0.2; visual box size=0.2 0.2 0.2
- added link act0Seg14helper_shape, mass 0.00035; collision cylinder length=0.2 radius=0.1; visual cylinder length=0.2 radius=0.1
- added link act0Seg15, mass 0.35; collision box size=0.2 0.2 0.2; visual box size=0.2 0.2 0.2
- added link act0Seg15helper_shape, mass 0.00035; collision cylinder length=0.2 radius=0.1; visual cylinder length=0.2 radius=0.1
- added link act0Seg16, mass 0.35; collision box size=0.2 0.2 0.2; visual box size=0.2 0.2 0.2
- added link act0Seg16helper_shape, mass 0.00035; collision cylinder length=0.2 radius=0.1; visual cylinder length=0.2 radius=0.1
- added link act0Seg17, mass 0.35; collision box size=0.2 0.2 0.2; visual box size=0.2 0.2 0.2
- added link act0Seg17helper_shape, mass 0.00035; collision cylinder length=0.2 radius=0.1; visual cylinder length=0.2 radius=0.1
- added link act0Seg18, mass 0.35; collision box size=0.2 0.2 0.2; visual box size=0.2 0.2 0.2
- added link act0Seg18helper_shape, mass 0.00035; collision cylinder length=0.2 radius=0.1; visual cylinder length=0.2 radius=0.1
- added link act0Seg19, mass 0.35; collision box size=0.2 0.2 0.2; visual box size=0.2 0.2 0.2
- added link act0Seg19helper_shape, mass 0.00035; collision cylinder length=0.2 radius=0.1; visual cylinder length=0.2 radius=0.1
- added link act0Seg20, mass 0.35; collision box size=0.2 0.2 0.1; visual box size=0.2 0.2 0.1
- added link act0Seg20helper_shape, mass 0.00035; collision cylinder length=0.2 radius=0.1; visual cylinder length=0.2 radius=0.1
- link act0Seg10: geometry collision box size=0.2 0.2 0.2; visual box size=0.2 0.2 0.2
Joints:
- added joint act0Seg10_to_act0Seg11_ax0: type revolute, parent act0Seg10, child act0Seg11, origin xyz=0.0 0.05 0.2 rpy=0.0 0.0 0.0, axis 1 0 0, limit lower=-3.141592 upper=3.141592 effort=100 velocity=3
- added joint act0Seg10_to_act0Seg11_ax0helper_shape: type fixed, parent act0Seg10, child act0Seg11helper_shape, origin xyz=0 0 0.2 rpy=0 0 0, axis 1 0 0
- added joint act0Seg11_to_act0Seg12_ax1: type revolute, parent act0Seg11, child act0Seg12, origin xyz=0.0 -0.05 0.2 rpy=0.0 0.0 0.0, axis 0 1 0, limit lower=-3.141592 upper=3.141592 effort=100 velocity=3
- added joint act0Seg11_to_act0Seg12_ax1helper_shape: type fixed, parent act0Seg11, child act0Seg12helper_shape, origin xyz=0.0 -0.05 0.2 rpy=0.0 0.0 0.0, axis 1 0 0
- added joint act0Seg12_to_act0Seg13_ax0: type revolute, parent act0Seg12, child act0Seg13, origin xyz=0.0 0.05 0.2 rpy=0.0 0.0 0.0, axis 1 0 0, limit lower=-3.141592 upper=3.141592 effort=100 velocity=3
- added joint act0Seg12_to_act0Seg13_ax0helper_shape: type fixed, parent act0Seg12, child act0Seg13helper_shape, origin xyz=0 0 0.2 rpy=0 0 0, axis 1 0 0
- added joint act0Seg13_to_act0Seg14_ax1: type revolute, parent act0Seg13, child act0Seg14, origin xyz=0.0 -0.05 0.2 rpy=0.0 0.0 0.0, axis 0 1 0, limit lower=-3.141592 upper=3.141592 effort=100 velocity=3
- added joint act0Seg13_to_act0Seg14_ax1helper_shape: type fixed, parent act0Seg13, child act0Seg14helper_shape, origin xyz=0.0 -0.05 0.2 rpy=0.0 0.0 0.0, axis 1 0 0
- added joint act0Seg14_to_act0Seg15_ax0: type revolute, parent act0Seg14, child act0Seg15, origin xyz=0.0 0.05 0.2 rpy=0.0 0.0 0.0, axis 1 0 0, limit lower=-3.141592 upper=3.141592 effort=100 velocity=3
- added joint act0Seg14_to_act0Seg15_ax0helper_shape: type fixed, parent act0Seg14, child act0Seg15helper_shape, origin xyz=0 0 0.2 rpy=0 0 0, axis 1 0 0
- added joint act0Seg15_to_act0Seg16_ax1: type revolute, parent act0Seg15, child act0Seg16, origin xyz=0.0 -0.05 0.2 rpy=0.0 0.0 0.0, axis 0 1 0, limit lower=-3.141592 upper=3.141592 effort=100 velocity=3
- added joint act0Seg15_to_act0Seg16_ax1helper_shape: type fixed, parent act0Seg15, child act0Seg16helper_shape, origin xyz=0.0 -0.05 0.2 rpy=0.0 0.0 0.0, axis 1 0 0
- added joint act0Seg16_to_act0Seg17_ax0: type revolute, parent act0Seg16, child act0Seg17, origin xyz=0.0 0.05 0.2 rpy=0.0 0.0 0.0, axis 1 0 0, limit lower=-3.141592 upper=3.141592 effort=100 velocity=3
- added joint act0Seg16_to_act0Seg17_ax0helper_shape: type fixed, parent act0Seg16, child act0Seg17helper_shape, origin xyz=0 0 0.2 rpy=0 0 0, axis 1 0 0
- added joint act0Seg17_to_act0Seg18_ax1: type revolute, parent act0Seg17, child act0Seg18, origin xyz=0.0 -0.05 0.2 rpy=0.0 0.0 0.0, axis 0 1 0, limit lower=-3.141592 upper=3.141592 effort=100 velocity=3
- added joint act0Seg17_to_act0Seg18_ax1helper_shape: type fixed, parent act0Seg17, child act0Seg18helper_shape, origin xyz=0.0 -0.05 0.2 rpy=0.0 0.0 0.0, axis 1 0 0
- added joint act0Seg18_to_act0Seg19_ax0: type revolute, parent act0Seg18, child act0Seg19, origin xyz=0.0 0.05 0.2 rpy=0.0 0.0 0.0, axis 1 0 0, limit lower=-3.141592 upper=3.141592 effort=100 velocity=3
- added joint act0Seg18_to_act0Seg19_ax0helper_shape: type fixed, parent act0Seg18, child act0Seg19helper_shape, origin xyz=0 0 0.2 rpy=0 0 0, axis 1 0 0
- added joint act0Seg19_to_act0Seg20_ax1: type revolute, parent act0Seg19, child act0Seg20, origin xyz=0.0 -0.05 0.2 rpy=0.0 0.0 0.0, axis 0 1 0, limit lower=-3.141592 upper=3.141592 effort=100 velocity=3
- added joint act0Seg19_to_act0Seg20_ax1helper_shape: type fixed, parent act0Seg19, child act0Seg20helper_shape, origin xyz=0.0 -0.05 0.2 rpy=0.0 0.0 0.0, axis 1 0 0
