Commit message: New updates

File: URDFS/box.urdf (robot description, URDF)
Before this commit: robot box, 1 links, 0 joints
Links:
- link box: geometry collision box size=1 100 2; visual box size=1 100 2
