Commit message: New updates

File: URDFS/cont_generated.urdf (robot description, URDF)
Before this commit: robot URDFS/cont_generated, 112 links, 111 joints
Links:
- added link act10Seg0, mass 0.00294; collision box size=1.0 1.0 0.25; visual box size=1.0 1.0 0.25
- added link act10Seg1, mass 0.00294; collision box size=1.0 1.0 0.5; visual box size=1.0 1.0 0.5
- added link act10Seg1helper_shape, mass 2.94e-06; collision cylinder length=1.0 radius=0.5; visual cylinder length=1.0 radius=0.5
- added link act10Seg2, mass 0.00294; collision box size=1.0 1.0 0.5; visual box size=1.0 1.0 0.5
- added link act10Seg2helper_shape, mass 2.94e-06; collision cylinder length=1.0 radius=0.5; visual cylinder length=1.0 radius=0.5
- added link act10Seg3, mass 0.00294; collision box size=1.0 1.0 0.5; visual box size=1.0 1.0 0.5
- added link act10Seg3helper_shape, mass 2.94e-06; collision cylinder length=1.0 radius=0.5; visual cylinder length=1.0 radius=0.5
- added link act10Seg4, mass 0.00294; collision box size=1.0 1.0 0.5; visual box size=1.0 1.0 0.5
- added link act10Seg4helper_shape, mass 2.94e-06; collision cylinder length=1.0 radius=0.5; visual cylinder length=1.0 radius=0.5
- added link act10Seg5, mass 0.00294; collision box size=1.0 1.0 0.25; visual box size=1.0 1.0 0.25
- added link act10Seg5helper_shape, mass 2.94e-06; collision cylinder length=1.0 radius=0.5; visual cylinder length=1.0 radius=0.5
- added link act11Seg0, mass 0.00294; collision box size=1.0 1.0 0.25; visual box size=1.0 1.0 0.25
- added link act11Seg1, mass 0.00294; collision box size=1.0 1.0 0.5; visual box size=1.0 1.0 0.5
- added link act11Seg1helper_shape, mass 2.94e-06; collision cylinder length=1.0 radius=0.5; visual cylinder length=1.0 radius=0.5
- added link act11Seg2, mass 0.00294; collision box size=1.0 1.0 0.5; visual box size=1.0 1.0 0.5
- added link act11Seg2helper_shape, mass 2.94e-06; collision cylinder length=1.0 radius=0.5; visual cylinder length=1.0 radius=0.5
- added link act11Seg3, mass 0.00294; collision box size=1.0 1.0 0.5; visual box size=1.0 1.0 0.5
- added link act11Seg3helper_shape, mass 2.94e-06; collision cylinder length=1.0 radius=0.5; visual cylinder length=1.0 radius=0.5
- added link act11Seg4, mass 0.00294; collision box size=1.0 1.0 0.5; visual box size=1.0 1.0 0.5
- added link act11Seg4helper_shape, mass 2.94e-06; collision cylinder length=1.0 radius=0.5; visual cylinder length=1.0 radius=0.5
- added link act11Seg5, mass 0.00294; collision box size=1.0 1.0 0.25; visual box size=1.0 1.0 0.25
- added link act11Seg5helper_shape, mass 2.94e-06; collision cylinder length=1.0 radius=0.5; visual cylinder length=1.0 radius=0.5
- added link act12Seg0, mass 0.00294; collision box size=1.0 1.0 0.25; visual box size=1.0 1.0 0.25
- added link act12Seg1, mass 0.00294; collision box size=1.0 1.0 0.5; visual box size=1.0 1.0 0.5
- added link act12Seg1helper_shape, mass 2.94e-06; collision cylinder length=1.0 radius=0.5; visual cylinder length=1.0 radius=0.5
- added link act12Seg2, mass 0.00294; collision box size=1.0 1.0 0.5; visual box size=1.0 1.0 0.5
- added link act12Seg2helper_shape, mass 2.94e-06; collision cylinder length=1.0 radius=0.5; visual cylinder length=1.0 radius=0.5
- added link act12Seg3, mass 0.00294; collision box size=1.0 1.0 0.5; visual box size=1.0 1.0 0.5
- added link act12Seg3helper_shape, mass 2.94e-06; collision cylinder length=1.0 radius=0.5; visual cylinder length=1.0 radius=0.5
- added link act12Seg4, mass 0.00294; collision box size=1.0 1.0 0.5; visual box size=1.0 1.0 0.5
- added link act12Seg4helper_shape, mass 2.94e-06; collision cylinder length=1.0 radius=0.5; visual cylinder length=1.0 radius=0.5
- added link act12Seg5, mass 0.00294; collision box size=1.0 1.0 0.25; visual box size=1.0 1.0 0.25
- added link act12Seg5helper_shape, mass 2.94e-06; collision cylinder length=1.0 radius=0.5; visual cylinder length=1.0 radius=0.5
- added link act13Seg0, mass 0.00294; collision box size=1.0 1.0 0.25; visual box size=1.0 1.0 0.25
- added link act13Seg1, mass 0.00294; collision box size=1.0 1.0 0.5; visual box size=1.0 1.0 0.5
- added link act13Seg1helper_shape, mass 2.94e-06; collision cylinder length=1.0 radius=0.5; visual cylinder length=1.0 radius=0.5
- added link act13Seg2, mass 0.00294; collision box size=1.0 1.0 0.5; visual box size=1.0 1.0 0.5
- added link act13Seg2helper_shape, mass 2.94e-06; collision cylinder length=1.0 radius=0.5; visual cylinder length=1.0 radius=0.5
- added link act13Seg3, mass 0.00294; collision box size=1.0 1.0 0.5; visual box size=1.0 1.0 0.5
- added link act13Seg3helper_shape, mass 2.94e-06; collision cylinder length=1.0 radius=0.5; visual cylinder length=1.0 radius=0.5
- added link act13Seg4, mass 0.00294; collision box size=1.0 1.0 0.5; visual box size=1.0 1.0 0.5
- added link act13Seg4helper_shape, mass 2.94e-06; collision cylinder length=1.0 radius=0.5; visual cylinder length=1.0 radius=0.5
- added link act13Seg5, mass 0.00294; collision box size=1.0 1.0 0.25; visual box size=1.0 1.0 0.25
- added link act13Seg5helper_shape, mass 2.94e-06; collision cylinder length=1.0 radius=0.5; visual cylinder length=1.0 radius=0.5
- added link act14Seg0, mass 0.00294; collision box size=1.0 1.0 0.25; visual box size=1.0 1.0 0.25
- added link act14Seg1, mass 0.00294; collision box size=1.0 1.0 0.5; visual box size=1.0 1.0 0.5
- added link act14Seg1helper_shape, mass 2.94e-06; collision cylinder length=1.0 radius=0.5; visual cylinder length=1.0 radius=0.5
- added link act14Seg2, mass 0.00294; collision box size=1.0 1.0 0.5; visual box size=1.0 1.0 0.5
- added link act14Seg2helper_shape, mass 2.94e-06; collision cylinder length=1.0 radius=0.5; visual cylinder length=1.0 radius=0.5
- added link act14Seg3, mass 0.00294; collision box size=1.0 1.0 0.5; visual box size=1.0 1.0 0.5
- added link act14Seg3helper_shape, mass 2.94e-06; collision cylinder length=1.0 radius=0.5; visual cylinder length=1.0 radius=0.5
- added link act14Seg4, mass 0.00294; collision box size=1.0 1.0 0.5; visual box size=1.0 1.0 0.5
- added link act14Seg4helper_shape, mass 2.94e-06; collision cylinder length=1.0 radius=0.5; visual cylinder length=1.0 radius=0.5
- added link act14Seg5, mass 0.00294; collision box size=1.0 1.0 0.25; visual box size=1.0 1.0 0.25
- added link act14Seg5helper_shape, mass 2.94e-06; collision cylinder length=1.0 radius=0.5; visual cylinder length=1.0 radius=0.5
- added link act15Seg0, mass 0.00294; collision box size=1.0 1.0 0.25; visual box size=1.0 1.0 0.25
- added link act15Seg1, mass 0.00294; collision box size=1.0 1.0 0.5; visual box size=1.0 1.0 0.5
- added link act15Seg1helper_shape, mass 2.94e-06; collision cylinder length=1.0 radius=0.5; visual cylinder length=1.0 radius=0.5
- added link act15Seg2, mass 0.00294; collision box size=1.0 1.0 0.5; visual box size=1.0 1.0 0.5
- added link act15Seg2helper_shape, mass 2.94e-06; collision cylinder length=1.0 radius=0.5; visual cylinder length=1.0 radius=0.5
- added link act15Seg3, mass 0.00294; collision box size=1.0 1.0 0.5; visual box size=1.0 1.0 0.5
- added link act15Seg3helper_shape, mass 2.94e-06; collision cylinder length=1.0 radius=0.5; visual cylinder length=1.0 radius=0.5
- added link act15Seg4, mass 0.00294; collision box size=1.0 1.0 0.5; visual box size=1.0 1.0 0.5
- added link act15Seg4helper_shape, mass 2.94e-06; collision cylinder length=1.0 radius=0.5; visual cylinder length=1.0 radius=0.5
- added link act15Seg5, mass 0.00294; collision box size=1.0 1.0 0.25; visual box size=1.0 1.0 0.25
- added link act15Seg5helper_shape, mass 2.94e-06; collision cylinder length=1.0 radius=0.5; visual cylinder length=1.0 radius=0.5
- added link act16Seg0, mass 0.00294; collision box size=1.0 1.0 0.25; visual box size=1.0 1.0 0.25
- added link act16Seg1, mass 0.00294; collision box size=1.0 1.0 0.5; visual box size=1.0 1.0 0.5
- added link act16Seg1helper_shape, mass 2.94e-06; collision cylinder length=1.0 radius=0.5; visual cylinder length=1.0 radius=0.5
- added link act16Seg2, mass 0.00294; collision box size=1.0 1.0 0.5; visual box size=1.0 1.0 0.5
- added link act16Seg2helper_shape, mass 2.94e-06; collision cylinder length=1.0 radius=0.5; visual cylinder length=1.0 radius=0.5
- added link act16Seg3, mass 0.00294; collision box size=1.0 1.0 0.5; visual box size=1.0 1.0 0.5
- added link act16Seg3helper_shape, mass 2.94e-06; collision cylinder length=1.0 radius=0.5; visual cylinder length=1.0 radius=0.5
- added link act16Seg4, mass 0.00294; collision box size=1.0 1.0 0.5; visual box size=1.0 1.0 0.5
- added link act16Seg4helper_shape, mass 2.94e-06; collision cylinder length=1.0 radius=0.5; visual cylinder length=1.0 radius=0.5
- added link act16Seg5, mass 0.00294; collision box size=1.0 1.0 0.25; visual box size=1.0 1.0 0.25
- added link act16Seg5helper_shape, mass 2.94e-06; collision cylinder length=1.0 radius=0.5; visual cylinder length=1.0 radius=0.5
- added link act17Seg0, mass 0.00294; collision box size=1.0 1.0 0.25; visual box size=1.0 1.0 0.25
- added link act17Seg1, mass 0.00294; collision box size=1.0 1.0 0.5; visual box size=1.0 1.0 0.5
- added link act17Seg1helper_shape, mass 2.94e-06; collision cylinder length=1.0 radius=0.5; visual cylinder length=1.0 radius=0.5
- added link act17Seg2, mass 0.00294; collision box size=1.0 1.0 0.5; visual box size=1.0 1.0 0.5
- added link act17Seg2helper_shape, mass 2.94e-06; collision cylinder length=1.0 radius=0.5; visual cylinder length=1.0 radius=0.5
- added link act17Seg3, mass 0.00294; collision box size=1.0 1.0 0.5; visual box size=1.0 1.0 0.5
- added link act17Seg3helper_shape, mass 2.94e-06; collision cylinder length=1.0 radius=0.5; visual cylinder length=1.0 radius=0.5
- added link act17Seg4, mass 0.00294; collision box size=1.0 1.0 0.5; visual box size=1.0 1.0 0.5
- added link act17Seg4helper_shape, mass 2.94e-06; collision cylinder length=1.0 radius=0.5; visual cylinder length=1.0 radius=0.5
- added link act17Seg5, mass 0.00294; collision box size=1.0 1.0 0.25; visual box size=1.0 1.0 0.25
- added link act17Seg5helper_shape, mass 2.94e-06; collision cylinder length=1.0 radius=0.5; visual cylinder length=1.0 radius=0.5
- added link act18Seg0, mass 0.00294; collision box size=1.0 1.0 0.25; visual box size=1.0 1.0 0.25
- added link act18Seg1, mass 0.00294; collision box size=1.0 1.0 0.5; visual box size=1.0 1.0 0.5
- added link act18Seg1helper_shape, mass 2.94e-06; collision cylinder length=1.0 radius=0.5; visual cylinder length=1.0 radius=0.5
- added link act18Seg2, mass 0.00294; collision box size=1.0 1.0 0.5; visual box size=1.0 1.0 0.5
- added link act18Seg2helper_shape, mass 2.94e-06; collision cylinder length=1.0 radius=0.5; visual cylinder length=1.0 radius=0.5
- added link act18Seg3, mass 0.00294; collision box size=1.0 1.0 0.5; visual box size=1.0 1.0 0.5
- added link act18Seg3helper_shape, mass 2.94e-06; collision cylinder length=1.0 radius=0.5; visual cylinder length=1.0 radius=0.5
- added link act18Seg4, mass 0.00294; collision box size=1.0 1.0 0.5; visual box size=1.0 1.0 0.5
- added link act18Seg4helper_shape, mass 2.94e-06; collision cylinder length=1.0 radius=0.5; visual cylinder length=1.0 radius=0.5
- added link act18Seg5, mass 0.00294; collision box size=1.0 1.0 0.25; visual box size=1.0 1.0 0.25
- added link act18Seg5helper_shape, mass 2.94e-06; collision cylinder length=1.0 radius=0.5; visual cylinder length=1.0 radius=0.5
- added link act19Seg0, mass 0.00294; collision box size=1.0 1.0 0.25; visual box size=1.0 1.0 0.25
- added link act19Seg1, mass 0.00294; collision box size=1.0 1.0 0.5; visual box size=1.0 1.0 0.5
- added link act19Seg1helper_shape, mass 2.94e-06; collision cylinder length=1.0 radius=0.5; visual cylinder length=1.0 radius=0.5
- added link act19Seg2, mass 0.00294; collision box size=1.0 1.0 0.5; visual box size=1.0 1.0 0.5
- added link act19Seg2helper_shape, mass 2.94e-06; collision cylinder length=1.0 radius=0.5; visual cylinder length=1.0 radius=0.5
- added link act19Seg3, mass 0.00294; collision box size=1.0 1.0 0.5; visual box size=1.0 1.0 0.5
- added link act19Seg3helper_shape, mass 2.94e-06; collision cylinder length=1.0 radius=0.5; visual cylinder length=1.0 radius=0.5
- added link act19Seg4, mass 0.00294; collision box size=1.0 1.0 0.5; visual box size=1.0 1.0 0.5
- added link act19Seg4helper_shape, mass 2.94e-06; collision cylinder length=1.0 radius=0.5; visual cylinder length=1.0 radius=0.5
- added link act19Seg5, mass 0.00294; collision box size=1.0 1.0 0.25; visual box size=1.0 1.0 0.25
- added link act19Seg5helper_shape, mass 2.94e-06; collision cylinder length=1.0 radius=0.5; visual cylinder length=1.0 radius=0.5
Joints:
- removed joint act9Seg5_to_tip_link0
- added joint act10Seg0_to_act10Seg1_ax0: type revolute, parent act10Seg0, child act10Seg1, origin xyz=0 0 0.25 rpy=0 0 0, axis 1 0 0, limit lower=-3.141592 upper=3.141592 effort=100 velocity=3
- added joint act10Seg0_to_act10Seg1_ax0helper_shape: type fixed, parent act10Seg0, child act10Seg1helper_shape, origin xyz=0 0 0.25 rpy=0 0 0, axis 1 0 0
- added joint act10Seg1_to_act10Seg2_ax0: type revolute, parent act10Seg1, child act10Seg2, origin xyz=0 0 0.5 rpy=0 0 0, axis 1 0 0, limit lower=-3.141592 upper=3.141592 effort=100 velocity=3
- added joint act10Seg1_to_act10Seg2_ax0helper_shape: type fixed, parent act10Seg1, child act10Seg2helper_shape, origin xyz=0 0 0.5 rpy=0 0 0, axis 1 0 0
- added joint act10Seg2_to_act10Seg3_ax0: type revolute, parent act10Seg2, child act10Seg3, origin xyz=0 0 0.5 rpy=0 0 0, axis 1 0 0, limit lower=-3.141592 upper=3.141592 effort=100 velocity=3
- added joint act10Seg2_to_act10Seg3_ax0helper_shape: type fixed, parent act10Seg2, child act10Seg3helper_shape, origin xyz=0 0 0.5 rpy=0 0 0, axis 1 0 0
- added joint act10Seg3_to_act10Seg4_ax0: type revolute, parent act10Seg3, child act10Seg4, origin xyz=0 0 0.5 rpy=0 0 0, axis 1 0 0, limit lower=-3.141592 upper=3.141592 effort=100 velocity=3
- added joint act10Seg3_to_act10Seg4_ax0helper_shape: type fixed, parent act10Seg3, child act10Seg4helper_shape, origin xyz=0 0 0.5 rpy=0 0 0, axis 1 0 0
- added joint act10Seg4_to_act10Seg5_ax0: type revolute, parent act10Seg4, child act10Seg5, origin xyz=0 0 0.5 rpy=0 0 0, axis 1 0 0, limit lower=-3.141592 upper=3.141592 effort=100 velocity=3
- added joint act10Seg4_to_act10Seg5_ax0helper_shape: type fixed, parent act10Seg4, child act10Seg5helper_shape, origin xyz=0 0 0.5 rpy=0 0 0, axis 1 0 0
- added joint act10Seg5_to_act11Seg0_ax0: type fixed, parent act10Seg5, child act11Seg0, origin xyz=0 0 0.25 rpy=0 0 0, axis 1 0 0, limit lower=-3.141592 upper=3.141592 effort=100 velocity=3
- added joint act11Seg0_to_act11Seg1_ax0: type revolute, parent act11Seg0, child act11Seg1, origin xyz=0 0 0.25 rpy=0 0 0, axis 1 0 0, limit lower=-3.141592 upper=3.141592 effort=100 velocity=3
- added joint act11Seg0_to_act11Seg1_ax0helper_shape: type fixed, parent act11Seg0, child act11Seg1helper_shape, origin xyz=0 0 0.25 rpy=0 0 0, axis 1 0 0
- added joint act11Seg1_to_act11Seg2_ax0: type revolute, parent act11Seg1, child act11Seg2, origin xyz=0 0 0.5 rpy=0 0 0, axis 1 0 0, limit lower=-3.141592 upper=3.141592 effort=100 velocity=3
- added joint act11Seg1_to_act11Seg2_ax0helper_shape: type fixed, parent act11Seg1, child act11Seg2helper_shape, origin xyz=0 0 0.5 rpy=0 0 0, axis 1 0 0
- added joint act11Seg2_to_act11Seg3_ax0: type revolute, parent act11Seg2, child act11Seg3, origin xyz=0 0 0.5 rpy=0 0 0, axis 1 0 0, limit lower=-3.141592 upper=3.141592 effort=100 velocity=3
- added joint act11Seg2_to_act11Seg3_ax0helper_shape: type fixed, parent act11Seg2, child act11Seg3helper_shape, origin xyz=0 0 0.5 rpy=0 0 0, axis 1 0 0
- added joint act11Seg3_to_act11Seg4_ax0: type revolute, parent act11Seg3, child act11Seg4, origin xyz=0 0 0.5 rpy=0 0 0, axis 1 0 0, limit lower=-3.141592 upper=3.141592 effort=100 velocity=3
- added joint act11Seg3_to_act11Seg4_ax0helper_shape: type fixed, parent act11Seg3, child act11Seg4helper_shape, origin xyz=0 0 0.5 rpy=0 0 0, axis 1 0 0
- added joint act11Seg4_to_act11Seg5_ax0: type revolute, parent act11Seg4, child act11Seg5, origin xyz=0 0 0.5 rpy=0 0 0, axis 1 0 0, limit lower=-3.141592 upper=3.141592 effort=100 velocity=3
- added joint act11Seg4_to_act11Seg5_ax0helper_shape: type fixed, parent act11Seg4, child act11Seg5helper_shape, origin xyz=0 0 0.5 rpy=0 0 0, axis 1 0 0
- added joint act11Seg5_to_act12Seg0_ax0: type fixed, parent act11Seg5, child act12Seg0, origin xyz=0 0 0.25 rpy=0 0 0, axis 1 0 0, limit lower=-3.141592 upper=3.141592 effort=100 velocity=3
- added joint act12Seg0_to_act12Seg1_ax0: type revolute, parent act12Seg0, child act12Seg1, origin xyz=0 0 0.25 rpy=0 0 0, axis 1 0 0, limit lower=-3.141592 upper=3.141592 effort=100 velocity=3
- added joint act12Seg0_to_act12Seg1_ax0helper_shape: type fixed, parent act12Seg0, child act12Seg1helper_shape, origin xyz=0 0 0.25 rpy=0 0 0, axis 1 0 0
- added joint act12Seg1_to_act12Seg2_ax0: type revolute, parent act12Seg1, child act12Seg2, origin xyz=0 0 0.5 rpy=0 0 0, axis 1 0 0, limit lower=-3.141592 upper=3.141592 effort=100 velocity=3
- added joint act12Seg1_to_act12Seg2_ax0helper_shape: type fixed, parent act12Seg1, child act12Seg2helper_shape, origin xyz=0 0 0.5 rpy=0 0 0, axis 1 0 0
- added joint act12Seg2_to_act12Seg3_ax0: type revolute, parent act12Seg2, child act12Seg3, origin xyz=0 0 0.5 rpy=0 0 0, axis 1 0 0, limit lower=-3.141592 upper=3.141592 effort=100 velocity=3
- added joint act12Seg2_to_act12Seg3_ax0helper_shape: type fixed, parent act12Seg2, child act12Seg3helper_shape, origin xyz=0 0 0.5 rpy=0 0 0, axis 1 0 0
- added joint act12Seg3_to_act12Seg4_ax0: type revolute, parent act12Seg3, child act12Seg4, origin xyz=0 0 0.5 rpy=0 0 0, axis 1 0 0, limit lower=-3.141592 upper=3.141592 effort=100 velocity=3
- added joint act12Seg3_to_act12Seg4_ax0helper_shape: type fixed, parent act12Seg3, child act12Seg4helper_shape, origin xyz=0 0 0.5 rpy=0 0 0, axis 1 0 0
- added joint act12Seg4_to_act12Seg5_ax0: type revolute, parent act12Seg4, child act12Seg5, origin xyz=0 0 0.5 rpy=0 0 0, axis 1 0 0, limit lower=-3.141592 upper=3.141592 effort=100 velocity=3
- added joint act12Seg4_to_act12Seg5_ax0helper_shape: type fixed, parent act12Seg4, child act12Seg5helper_shape, origin xyz=0 0 0.5 rpy=0 0 0, axis 1 0 0
- added joint act12Seg5_to_act13Seg0_ax0: type fixed, parent act12Seg5, child act13Seg0, origin xyz=0 0 0.25 rpy=0 0 0, axis 1 0 0, limit lower=-3.141592 upper=3.141592 effort=100 velocity=3
- added joint act13Seg0_to_act13Seg1_ax0: type revolute, parent act13Seg0, child act13Seg1, origin xyz=0 0 0.25 rpy=0 0 0, axis 1 0 0, limit lower=-3.141592 upper=3.141592 effort=100 velocity=3
- added joint act13Seg0_to_act13Seg1_ax0helper_shape: type fixed, parent act13Seg0, child act13Seg1helper_shape, origin xyz=0 0 0.25 rpy=0 0 0, axis 1 0 0
- added joint act13Seg1_to_act13Seg2_ax0: type revolute, parent act13Seg1, child act13Seg2, origin xyz=0 0 0.5 rpy=0 0 0, axis 1 0 0, limit lower=-3.141592 upper=3.141592 effort=100 velocity=3
- added joint act13Seg1_to_act13Seg2_ax0helper_shape: type fixed, parent act13Seg1, child act13Seg2helper_shape, origin xyz=0 0 0.5 rpy=0 0 0, axis 1 0 0
- added joint act13Seg2_to_act13Seg3_ax0: type revolute, parent act13Seg2, child act13Seg3, origin xyz=0 0 0.5 rpy=0 0 0, axis 1 0 0, limit lower=-3.141592 upper=3.141592 effort=100 velocity=3
- added joint act13Seg2_to_act13Seg3_ax0helper_shape: type fixed, parent act13Seg2, child act13Seg3helper_shape, origin xyz=0 0 0.5 rpy=0 0 0, axis 1 0 0
- added joint act13Seg3_to_act13Seg4_ax0: type revolute, parent act13Seg3, child act13Seg4, origin xyz=0 0 0.5 rpy=0 0 0, axis 1 0 0, limit lower=-3.141592 upper=3.141592 effort=100 velocity=3
- added joint act13Seg3_to_act13Seg4_ax0helper_shape: type fixed, parent act13Seg3, child act13Seg4helper_shape, origin xyz=0 0 0.5 rpy=0 0 0, axis 1 0 0
- added joint act13Seg4_to_act13Seg5_ax0: type revolute, parent act13Seg4, child act13Seg5, origin xyz=0 0 0.5 rpy=0 0 0, axis 1 0 0, limit lower=-3.141592 upper=3.141592 effort=100 velocity=3
- added joint act13Seg4_to_act13Seg5_ax0helper_shape: type fixed, parent act13Seg4, child act13Seg5helper_shape, origin xyz=0 0 0.5 rpy=0 0 0, axis 1 0 0
- added joint act13Seg5_to_act14Seg0_ax0: type fixed, parent act13Seg5, child act14Seg0, origin xyz=0 0 0.25 rpy=0 0 0, axis 1 0 0, limit lower=-3.141592 upper=3.141592 effort=100 velocity=3
- added joint act14Seg0_to_act14Seg1_ax0: type revolute, parent act14Seg0, child act14Seg1, origin xyz=0 0 0.25 rpy=0 0 0, axis 1 0 0, limit lower=-3.141592 upper=3.141592 effort=100 velocity=3
- added joint act14Seg0_to_act14Seg1_ax0helper_shape: type fixed, parent act14Seg0, child act14Seg1helper_shape, origin xyz=0 0 0.25 rpy=0 0 0, axis 1 0 0
- added joint act14Seg1_to_act14Seg2_ax0: type revolute, parent act14Seg1, child act14Seg2, origin xyz=0 0 0.5 rpy=0 0 0, axis 1 0 0, limit lower=-3.141592 upper=3.141592 effort=100 velocity=3
- added joint act14Seg1_to_act14Seg2_ax0helper_shape: type fixed, parent act14Seg1, child act14Seg2helper_shape, origin xyz=0 0 0.5 rpy=0 0 0, axis 1 0 0
- added joint act14Seg2_to_act14Seg3_ax0: type revolute, parent act14Seg2, child act14Seg3, origin xyz=0 0 0.5 rpy=0 0 0, axis 1 0 0, limit lower=-3.141592 upper=3.141592 effort=100 velocity=3
- added joint act14Seg2_to_act14Seg3_ax0helper_shape: type fixed, parent act14Seg2, child act14Seg3helper_shape, origin xyz=0 0 0.5 rpy=0 0 0, axis 1 0 0
- added joint act14Seg3_to_act14Seg4_ax0: type revolute, parent act14Seg3, child act14Seg4, origin xyz=0 0 0.5 rpy=0 0 0, axis 1 0 0, limit lower=-3.141592 upper=3.141592 effort=100 velocity=3
- added joint act14Seg3_to_act14Seg4_ax0helper_shape: type fixed, parent act14Seg3, child act14Seg4helper_shape, origin xyz=0 0 0.5 rpy=0 0 0, axis 1 0 0
- added joint act14Seg4_to_act14Seg5_ax0: type revolute, parent act14Seg4, child act14Seg5, origin xyz=0 0 0.5 rpy=0 0 0, axis 1 0 0, limit lower=-3.141592 upper=3.141592 effort=100 velocity=3
- added joint act14Seg4_to_act14Seg5_ax0helper_shape: type fixed, parent act14Seg4, child act14Seg5helper_shape, origin xyz=0 0 0.5 rpy=0 0 0, axis 1 0 0
- added joint act14Seg5_to_act15Seg0_ax0: type fixed, parent act14Seg5, child act15Seg0, origin xyz=0 0 0.25 rpy=0 0 0, axis 1 0 0, limit lower=-3.141592 upper=3.141592 effort=100 velocity=3
- added joint act15Seg0_to_act15Seg1_ax0: type revolute, parent act15Seg0, child act15Seg1, origin xyz=0 0 0.25 rpy=0 0 0, axis 1 0 0, limit lower=-3.141592 upper=3.141592 effort=100 velocity=3
- added joint act15Seg0_to_act15Seg1_ax0helper_shape: type fixed, parent act15Seg0, child act15Seg1helper_shape, origin xyz=0 0 0.25 rpy=0 0 0, axis 1 0 0
- added joint act15Seg1_to_act15Seg2_ax0: type revolute, parent act15Seg1, child act15Seg2, origin xyz=0 0 0.5 rpy=0 0 0, axis 1 0 0, limit lower=-3.141592 upper=3.141592 effort=100 velocity=3
- added joint act15Seg1_to_act15Seg2_ax0helper_shape: type fixed, parent act15Seg1, child act15Seg2helper_shape, origin xyz=0 0 0.5 rpy=0 0 0, axis 1 0 0
- added joint act15Seg2_to_act15Seg3_ax0: type revolute, parent act15Seg2, child act15Seg3, origin xyz=0 0 0.5 rpy=0 0 0, axis 1 0 0, limit lower=-3.141592 upper=3.141592 effort=100 velocity=3
- added joint act15Seg2_to_act15Seg3_ax0helper_shape: type fixed, parent act15Seg2, child act15Seg3helper_shape, origin xyz=0 0 0.5 rpy=0 0 0, axis 1 0 0
- added joint act15Seg3_to_act15Seg4_ax0: type revolute, parent act15Seg3, child act15Seg4, origin xyz=0 0 0.5 rpy=0 0 0, axis 1 0 0, limit lower=-3.141592 upper=3.141592 effort=100 velocity=3
- added joint act15Seg3_to_act15Seg4_ax0helper_shape: type fixed, parent act15Seg3, child act15Seg4helper_shape, origin xyz=0 0 0.5 rpy=0 0 0, axis 1 0 0
- added joint act15Seg4_to_act15Seg5_ax0: type revolute, parent act15Seg4, child act15Seg5, origin xyz=0 0 0.5 rpy=0 0 0, axis 1 0 0, limit lower=-3.141592 upper=3.141592 effort=100 velocity=3
- added joint act15Seg4_to_act15Seg5_ax0helper_shape: type fixed, parent act15Seg4, child act15Seg5helper_shape, origin xyz=0 0 0.5 rpy=0 0 0, axis 1 0 0
- added joint act15Seg5_to_act16Seg0_ax0: type fixed, parent act15Seg5, child act16Seg0, origin xyz=0 0 0.25 rpy=0 0 0, axis 1 0 0, limit lower=-3.141592 upper=3.141592 effort=100 velocity=3
- added joint act16Seg0_to_act16Seg1_ax0: type revolute, parent act16Seg0, child act16Seg1, origin xyz=0 0 0.25 rpy=0 0 0, axis 1 0 0, limit lower=-3.141592 upper=3.141592 effort=100 velocity=3
- added joint act16Seg0_to_act16Seg1_ax0helper_shape: type fixed, parent act16Seg0, child act16Seg1helper_shape, origin xyz=0 0 0.25 rpy=0 0 0, axis 1 0 0
- added joint act16Seg1_to_act16Seg2_ax0: type revolute, parent act16Seg1, child act16Seg2, origin xyz=0 0 0.5 rpy=0 0 0, axis 1 0 0, limit lower=-3.141592 upper=3.141592 effort=100 velocity=3
- added joint act16Seg1_to_act16Seg2_ax0helper_shape: type fixed, parent act16Seg1, child act16Seg2helper_shape, origin xyz=0 0 0.5 rpy=0 0 0, axis 1 0 0
- added joint act16Seg2_to_act16Seg3_ax0: type revolute, parent act16Seg2, child act16Seg3, origin xyz=0 0 0.5 rpy=0 0 0, axis 1 0 0, limit lower=-3.141592 upper=3.141592 effort=100 velocity=3
- added joint act16Seg2_to_act16Seg3_ax0helper_shape: type fixed, parent act16Seg2, child act16Seg3helper_shape, origin xyz=0 0 0.5 rpy=0 0 0, axis 1 0 0
- added joint act16Seg3_to_act16Seg4_ax0: type revolute, parent act16Seg3, child act16Seg4, origin xyz=0 0 0.5 rpy=0 0 0, axis 1 0 0, limit lower=-3.141592 upper=3.141592 effort=100 velocity=3
- added joint act16Seg3_to_act16Seg4_ax0helper_shape: type fixed, parent act16Seg3, child act16Seg4helper_shape, origin xyz=0 0 0.5 rpy=0 0 0, axis 1 0 0
- added joint act16Seg4_to_act16Seg5_ax0: type revolute, parent act16Seg4, child act16Seg5, origin xyz=0 0 0.5 rpy=0 0 0, axis 1 0 0, limit lower=-3.141592 upper=3.141592 effort=100 velocity=3
- added joint act16Seg4_to_act16Seg5_ax0helper_shape: type fixed, parent act16Seg4, child act16Seg5helper_shape, origin xyz=0 0 0.5 rpy=0 0 0, axis 1 0 0
- added joint act16Seg5_to_act17Seg0_ax0: type fixed, parent act16Seg5, child act17Seg0, origin xyz=0 0 0.25 rpy=0 0 0, axis 1 0 0, limit lower=-3.141592 upper=3.141592 effort=100 velocity=3
- added joint act17Seg0_to_act17Seg1_ax0: type revolute, parent act17Seg0, child act17Seg1, origin xyz=0 0 0.25 rpy=0 0 0, axis 1 0 0, limit lower=-3.141592 upper=3.141592 effort=100 velocity=3
- added joint act17Seg0_to_act17Seg1_ax0helper_shape: type fixed, parent act17Seg0, child act17Seg1helper_shape, origin xyz=0 0 0.25 rpy=0 0 0, axis 1 0 0
- added joint act17Seg1_to_act17Seg2_ax0: type revolute, parent act17Seg1, child act17Seg2, origin xyz=0 0 0.5 rpy=0 0 0, axis 1 0 0, limit lower=-3.141592 upper=3.141592 effort=100 velocity=3
- added joint act17Seg1_to_act17Seg2_ax0helper_shape: type fixed, parent act17Seg1, child act17Seg2helper_shape, origin xyz=0 0 0.5 rpy=0 0 0, axis 1 0 0
- added joint act17Seg2_to_act17Seg3_ax0: type revolute, parent act17Seg2, child act17Seg3, origin xyz=0 0 0.5 rpy=0 0 0, axis 1 0 0, limit lower=-3.141592 upper=3.141592 effort=100 velocity=3
- added joint act17Seg2_to_act17Seg3_ax0helper_shape: type fixed, parent act17Seg2, child act17Seg3helper_shape, origin xyz=0 0 0.5 rpy=0 0 0, axis 1 0 0
- added joint act17Seg3_to_act17Seg4_ax0: type revolute, parent act17Seg3, child act17Seg4, origin xyz=0 0 0.5 rpy=0 0 0, axis 1 0 0, limit lower=-3.141592 upper=3.141592 effort=100 velocity=3
- added joint act17Seg3_to_act17Seg4_ax0helper_shape: type fixed, parent act17Seg3, child act17Seg4helper_shape, origin xyz=0 0 0.5 rpy=0 0 0, axis 1 0 0
- added joint act17Seg4_to_act17Seg5_ax0: type revolute, parent act17Seg4, child act17Seg5, origin xyz=0 0 0.5 rpy=0 0 0, axis 1 0 0, limit lower=-3.141592 upper=3.141592 effort=100 velocity=3
- added joint act17Seg4_to_act17Seg5_ax0helper_shape: type fixed, parent act17Seg4, child act17Seg5helper_shape, origin xyz=0 0 0.5 rpy=0 0 0, axis 1 0 0
- added joint act17Seg5_to_act18Seg0_ax0: type fixed, parent act17Seg5, child act18Seg0, origin xyz=0 0 0.25 rpy=0 0 0, axis 1 0 0, limit lower=-3.141592 upper=3.141592 effort=100 velocity=3
- added joint act18Seg0_to_act18Seg1_ax0: type revolute, parent act18Seg0, child act18Seg1, origin xyz=0 0 0.25 rpy=0 0 0, axis 1 0 0, limit lower=-3.141592 upper=3.141592 effort=100 velocity=3
- added joint act18Seg0_to_act18Seg1_ax0helper_shape: type fixed, parent act18Seg0, child act18Seg1helper_shape, origin xyz=0 0 0.25 rpy=0 0 0, axis 1 0 0
- added joint act18Seg1_to_act18Seg2_ax0: type revolute, parent act18Seg1, child act18Seg2, origin xyz=0 0 0.5 rpy=0 0 0, axis 1 0 0, limit lower=-3.141592 upper=3.141592 effort=100 velocity=3
- added joint act18Seg1_to_act18Seg2_ax0helper_shape: type fixed, parent act18Seg1, child act18Seg2helper_shape, origin xyz=0 0 0.5 rpy=0 0 0, axis 1 0 0
- added joint act18Seg2_to_act18Seg3_ax0: type revolute, parent act18Seg2, child act18Seg3, origin xyz=0 0 0.5 rpy=0 0 0, axis 1 0 0, limit lower=-3.141592 upper=3.141592 effort=100 velocity=3
- added joint act18Seg2_to_act18Seg3_ax0helper_shape: type fixed, parent act18Seg2, child act18Seg3helper_shape, origin xyz=0 0 0.5 rpy=0 0 0, axis 1 0 0
- added joint act18Seg3_to_act18Seg4_ax0: type revolute, parent act18Seg3, child act18Seg4, origin xyz=0 0 0.5 rpy=0 0 0, axis 1 0 0, limit lower=-3.141592 upper=3.141592 effort=100 velocity=3
- added joint act18Seg3_to_act18Seg4_ax0helper_shape: type fixed, parent act18Seg3, child act18Seg4helper_shape, origin xyz=0 0 0.5 rpy=0 0 0, axis 1 0 0
- added joint act18Seg4_to_act18Seg5_ax0: type revolute, parent act18Seg4, child act18Seg5, origin xyz=0 0 0.5 rpy=0 0 0, axis 1 0 0, limit lower=-3.141592 upper=3.141592 effort=100 velocity=3
- added joint act18Seg4_to_act18Seg5_ax0helper_shape: type fixed, parent act18Seg4, child act18Seg5helper_shape, origin xyz=0 0 0.5 rpy=0 0 0, axis 1 0 0
- added joint act18Seg5_to_act19Seg0_ax0: type fixed, parent act18Seg5, child act19Seg0, origin xyz=0 0 0.25 rpy=0 0 0, axis 1 0 0, limit lower=-3.141592 upper=3.141592 effort=100 velocity=3
- added joint act19Seg0_to_act19Seg1_ax0: type revolute, parent act19Seg0, child act19Seg1, origin xyz=0 0 0.25 rpy=0 0 0, axis 1 0 0, limit lower=-3.141592 upper=3.141592 effort=100 velocity=3
- added joint act19Seg0_to_act19Seg1_ax0helper_shape: type fixed, parent act19Seg0, child act19Seg1helper_shape, origin xyz=0 0 0.25 rpy=0 0 0, axis 1 0 0
- added joint act19Seg1_to_act19Seg2_ax0: type revolute, parent act19Seg1, child act19Seg2, origin xyz=0 0 0.5 rpy=0 0 0, axis 1 0 0, limit lower=-3.141592 upper=3.141592 effort=100 velocity=3
- added joint act19Seg1_to_act19Seg2_ax0helper_shape: type fixed, parent act19Seg1, child act19Seg2helper_shape, origin xyz=0 0 0.5 rpy=0 0 0, axis 1 0 0
- added joint act19Seg2_to_act19Seg3_ax0: type revolute, parent act19Seg2, child act19Seg3, origin xyz=0 0 0.5 rpy=0 0 0, axis 1 0 0, limit lower=-3.141592 upper=3.141592 effort=100 velocity=3
- added joint act19Seg2_to_act19Seg3_ax0helper_shape: type fixed, parent act19Seg2, child act19Seg3helper_shape, origin xyz=0 0 0.5 rpy=0 0 0, axis 1 0 0
- added joint act19Seg3_to_act19Seg4_ax0: type revolute, parent act19Seg3, child act19Seg4, origin xyz=0 0 0.5 rpy=0 0 0, axis 1 0 0, limit lower=-3.141592 upper=3.141592 effort=100 velocity=3
- added joint act19Seg3_to_act19Seg4_ax0helper_shape: type fixed, parent act19Seg3, child act19Seg4helper_shape, origin xyz=0 0 0.5 rpy=0 0 0, axis 1 0 0
- added joint act19Seg4_to_act19Seg5_ax0: type revolute, parent act19Seg4, child act19Seg5, origin xyz=0 0 0.5 rpy=0 0 0, axis 1 0 0, limit lower=-3.141592 upper=3.141592 effort=100 velocity=3
- added joint act19Seg4_to_act19Seg5_ax0helper_shape: type fixed, parent act19Seg4, child act19Seg5helper_shape, origin xyz=0 0 0.5 rpy=0 0 0, axis 1 0 0
- added joint act19Seg5_to_tip_link0: type fixed, parent act19Seg5, child tip_link0, origin xyz=0 0 0.25 rpy=0 0 0, axis 1 0 0
- added joint act9Seg5_to_act10Seg0_ax0: type fixed, parent act9Seg5, child act10Seg0, origin xyz=0 0 0.25 rpy=0 0 0, axis 1 0 0, limit lower=-3.141592 upper=3.141592 effort=100 velocity=3
