Commit message: Added obstacle GUI

File: URDFS/cont_generated.urdf (robot description, URDF)
Before this commit: robot URDFS/cont_generated, 222 links, 221 joints
Links:
- link act0Seg0: mass 0.00294 -> 0.294
- link act0Seg1: mass 0.00294 -> 0.294
- link act0Seg1helper_shape: mass 2.94e-06 -> 0.000294
- link act0Seg2: mass 0.00294 -> 0.294
- link act0Seg2helper_shape: mass 2.94e-06 -> 0.000294
- link act0Seg3: mass 0.00294 -> 0.294
- link act0Seg3helper_shape: mass 2.94e-06 -> 0.000294
- link act0Seg4: mass 0.00294 -> 0.294
- link act0Seg4helper_shape: mass 2.94e-06 -> 0.000294
- link act0Seg5: mass 0.00294 -> 0.294
- link act0Seg5helper_shape: mass 2.94e-06 -> 0.000294
- link act10Seg0: mass 0.00294 -> 0.294
- link act10Seg1: mass 0.00294 -> 0.294
- link act10Seg1helper_shape: mass 2.94e-06 -> 0.000294
- link act10Seg2: mass 0.00294 -> 0.294
- link act10Seg2helper_shape: mass 2.94e-06 -> 0.000294
- link act10Seg3: mass 0.00294 -> 0.294
- link act10Seg3helper_shape: mass 2.94e-06 -> 0.000294
- link act10Seg4: mass 0.00294 -> 0.294
- link act10Seg4helper_shape: mass 2.94e-06 -> 0.000294
- link act10Seg5: mass 0.00294 -> 0.294
- link act10Seg5helper_shape: mass 2.94e-06 -> 0.000294
- link act11Seg0: mass 0.00294 -> 0.294
- link act11Seg1: mass 0.00294 -> 0.294
- link act11Seg1helper_shape: mass 2.94e-06 -> 0.000294
- link act11Seg2: mass 0.00294 -> 0.294
- link act11Seg2helper_shape: mass 2.94e-06 -> 0.000294
- link act11Seg3: mass 0.00294 -> 0.294
- link act11Seg3helper_shape: mass 2.94e-06 -> 0.000294
- link act11Seg4: mass 0.00294 -> 0.294
- link act11Seg4helper_shape: mass 2.94e-06 -> 0.000294
- link act11Seg5: mass 0.00294 -> 0.294
- link act11Seg5helper_shape: mass 2.94e-06 -> 0.000294
- link act12Seg0: mass 0.00294 -> 0.294
- link act12Seg1: mass 0.00294 -> 0.294
- link act12Seg1helper_shape: mass 2.94e-06 -> 0.000294
- link act12Seg2: mass 0.00294 -> 0.294
- link act12Seg2helper_shape: mass 2.94e-06 -> 0.000294
- link act12Seg3: mass 0.00294 -> 0.294
- link act12Seg3helper_shape: mass 2.94e-06 -> 0.000294
- link act12Seg4: mass 0.00294 -> 0.294
- link act12Seg4helper_shape: mass 2.94e-06 -> 0.000294
- link act12Seg5: mass 0.00294 -> 0.294
- link act12Seg5helper_shape: mass 2.94e-06 -> 0.000294
- link act13Seg0: mass 0.00294 -> 0.294
- link act13Seg1: mass 0.00294 -> 0.294
- link act13Seg1helper_shape: mass 2.94e-06 -> 0.000294
- link act13Seg2: mass 0.00294 -> 0.294
- link act13Seg2helper_shape: mass 2.94e-06 -> 0.000294
- link act13Seg3: mass 0.00294 -> 0.294
- link act13Seg3helper_shape: mass 2.94e-06 -> 0.000294
- link act13Seg4: mass 0.00294 -> 0.294
- link act13Seg4helper_shape: mass 2.94e-06 -> 0.000294
- link act13Seg5: mass 0.00294 -> 0.294
- link act13Seg5helper_shape: mass 2.94e-06 -> 0.000294
- link act14Seg0: mass 0.00294 -> 0.294
- link act14Seg1: mass 0.00294 -> 0.294
- link act14Seg1helper_shape: mass 2.94e-06 -> 0.000294
- link act14Seg2: mass 0.00294 -> 0.294
- link act14Seg2helper_shape: mass 2.94e-06 -> 0.000294
- link act14Seg3: mass 0.00294 -> 0.294
- link act14Seg3helper_shape: mass 2.94e-06 -> 0.000294
- link act14Seg4: mass 0.00294 -> 0.294
- link act14Seg4helper_shape: mass 2.94e-06 -> 0.000294
- link act14Seg5: mass 0.00294 -> 0.294
- link act14Seg5helper_shape: mass 2.94e-06 -> 0.000294
- link act15Seg0: mass 0.00294 -> 0.294
- link act15Seg1: mass 0.00294 -> 0.294
- link act15Seg1helper_shape: mass 2.94e-06 -> 0.000294
- link act15Seg2: mass 0.00294 -> 0.294
- link act15Seg2helper_shape: mass 2.94e-06 -> 0.000294
- link act15Seg3: mass 0.00294 -> 0.294
- link act15Seg3helper_shape: mass 2.94e-06 -> 0.000294
- link act15Seg4: mass 0.00294 -> 0.294
- link act15Seg4helper_shape: mass 2.94e-06 -> 0.000294
- link act15Seg5: mass 0.00294 -> 0.294
- link act15Seg5helper_shape: mass 2.94e-06 -> 0.000294
- link act16Seg0: mass 0.00294 -> 0.294
- link act16Seg1: mass 0.00294 -> 0.294
- link act16Seg1helper_shape: mass 2.94e-06 -> 0.000294
- link act16Seg2: mass 0.00294 -> 0.294
- link act16Seg2helper_shape: mass 2.94e-06 -> 0.000294
- link act16Seg3: mass 0.00294 -> 0.294
- link act16Seg3helper_shape: mass 2.94e-06 -> 0.000294
- link act16Seg4: mass 0.00294 -> 0.294
- link act16Seg4helper_shape: mass 2.94e-06 -> 0.000294
- link act16Seg5: mass 0.00294 -> 0.294
- link act16Seg5helper_shape: mass 2.94e-06 -> 0.000294
- link act17Seg0: mass 0.00294 -> 0.294
- link act17Seg1: mass 0.00294 -> 0.294
- link act17Seg1helper_shape: mass 2.94e-06 -> 0.000294
- link act17Seg2: mass 0.00294 -> 0.294
- link act17Seg2helper_shape: mass 2.94e-06 -> 0.000294
- link act17Seg3: mass 0.00294 -> 0.294
- link act17Seg3helper_shape: mass 2.94e-06 -> 0.000294
- link act17Seg4: mass 0.00294 -> 0.294
- link act17Seg4helper_shape: mass 2.94e-06 -> 0.000294
- link act17Seg5: mass 0.00294 -> 0.294
- link act17Seg5helper_shape: mass 2.94e-06 -> 0.000294
- link act18Seg0: mass 0.00294 -> 0.294
- link act18Seg1: mass 0.00294 -> 0.294
- link act18Seg1helper_shape: mass 2.94e-06 -> 0.000294
- link act18Seg2: mass 0.00294 -> 0.294
- link act18Seg2helper_shape: mass 2.94e-06 -> 0.000294
- link act18Seg3: mass 0.00294 -> 0.294
- link act18Seg3helper_shape: mass 2.94e-06 -> 0.000294
- link act18Seg4: mass 0.00294 -> 0.294
- link act18Seg4helper_shape: mass 2.94e-06 -> 0.000294
- link act18Seg5: mass 0.00294 -> 0.294
- link act18Seg5helper_shape: mass 2.94e-06 -> 0.000294
- link act19Seg0: mass 0.00294 -> 0.294
- link act19Seg1: mass 0.00294 -> 0.294
- link act19Seg1helper_shape: mass 2.94e-06 -> 0.000294
- link act19Seg2: mass 0.00294 -> 0.294
- link act19Seg2helper_shape: mass 2.94e-06 -> 0.000294
- link act19Seg3: mass 0.00294 -> 0.294
- link act19Seg3helper_shape: mass 2.94e-06 -> 0.000294
- link act19Seg4: mass 0.00294 -> 0.294
- link act19Seg4helper_shape: mass 2.94e-06 -> 0.000294
- link act19Seg5: mass 0.00294 -> 0.294
- link act19Seg5helper_shape: mass 2.94e-06 -> 0.000294
- link act1Seg0: mass 0.00294 -> 0.294
- link act1Seg1: mass 0.00294 -> 0.294
- link act1Seg1helper_shape: mass 2.94e-06 -> 0.000294
- link act1Seg2: mass 0.00294 -> 0.294
- link act1Seg2helper_shape: mass 2.94e-06 -> 0.000294
- link act1Seg3: mass 0.00294 -> 0.294
- link act1Seg3helper_shape: mass 2.94e-06 -> 0.000294
- link act1Seg4: mass 0.00294 -> 0.294
- link act1Seg4helper_shape: mass 2.94e-06 -> 0.000294
- link act1Seg5: mass 0.00294 -> 0.294
- link act1Seg5helper_shape: mass 2.94e-06 -> 0.000294
- link act2Seg0: mass 0.00294 -> 0.294
- link act2Seg1: mass 0.00294 -> 0.294
- link act2Seg1helper_shape: mass 2.94e-06 -> 0.000294
- link act2Seg2: mass 0.00294 -> 0.294
- link act2Seg2helper_shape: mass 2.94e-06 -> 0.000294
- link act2Seg3: mass 0.00294 -> 0.294
- link act2Seg3helper_shape: mass 2.94e-06 -> 0.000294
- link act2Seg4: mass 0.00294 -> 0.294
- link act2Seg4helper_shape: mass 2.94e-06 -> 0.000294
- link act2Seg5: mass 0.00294 -> 0.294
- link act2Seg5helper_shape: mass 2.94e-06 -> 0.000294
- link act3Seg0: mass 0.00294 -> 0.294
- link act3Seg1: mass 0.00294 -> 0.294
- link act3Seg1helper_shape: mass 2.94e-06 -> 0.000294
- link act3Seg2: mass 0.00294 -> 0.294
- link act3Seg2helper_shape: mass 2.94e-06 -> 0.000294
- link act3Seg3: mass 0.00294 -> 0.294
- link act3Seg3helper_shape: mass 2.94e-06 -> 0.000294
- link act3Seg4: mass 0.00294 -> 0.294
- link act3Seg4helper_shape: mass 2.94e-06 -> 0.000294
- link act3Seg5: mass 0.00294 -> 0.294
- link act3Seg5helper_shape: mass 2.94e-06 -> 0.000294
- link act4Seg0: mass 0.00294 -> 0.294
- link act4Seg1: mass 0.00294 -> 0.294
- link act4Seg1helper_shape: mass 2.94e-06 -> 0.000294
- link act4Seg2: mass 0.00294 -> 0.294
- link act4Seg2helper_shape: mass 2.94e-06 -> 0.000294
- link act4Seg3: mass 0.00294 -> 0.294
- link act4Seg3helper_shape: mass 2.94e-06 -> 0.000294
- link act4Seg4: mass 0.00294 -> 0.294
- link act4Seg4helper_shape: mass 2.94e-06 -> 0.000294
- link act4Seg5: mass 0.00294 -> 0.294
- link act4Seg5helper_shape: mass 2.94e-06 -> 0.000294
- link act5Seg0: mass 0.00294 -> 0.294
- link act5Seg1: mass 0.00294 -> 0.294
- link act5Seg1helper_shape: mass 2.94e-06 -> 0.000294
- link act5Seg2: mass 0.00294 -> 0.294
- link act5Seg2helper_shape: mass 2.94e-06 -> 0.000294
- link act5Seg3: mass 0.00294 -> 0.294
- link act5Seg3helper_shape: mass 2.94e-06 -> 0.000294
- link act5Seg4: mass 0.00294 -> 0.294
- link act5Seg4helper_shape: mass 2.94e-06 -> 0.000294
- link act5Seg5: mass 0.00294 -> 0.294
- link act5Seg5helper_shape: mass 2.94e-06 -> 0.000294
- link act6Seg0: mass 0.00294 -> 0.294
- link act6Seg1: mass 0.00294 -> 0.294
- link act6Seg1helper_shape: mass 2.94e-06 -> 0.000294
- link act6Seg2: mass 0.00294 -> 0.294
- link act6Seg2helper_shape: mass 2.94e-06 -> 0.000294
- link act6Seg3: mass 0.00294 -> 0.294
- link act6Seg3helper_shape: mass 2.94e-06 -> 0.000294
- link act6Seg4: mass 0.00294 -> 0.294
- link act6Seg4helper_shape: mass 2.94e-06 -> 0.000294
- link act6Seg5: mass 0.00294 -> 0.294
- link act6Seg5helper_shape: mass 2.94e-06 -> 0.000294
- link act7Seg0: mass 0.00294 -> 0.294
- link act7Seg1: mass 0.00294 -> 0.294
- link act7Seg1helper_shape: mass 2.94e-06 -> 0.000294
- link act7Seg2: mass 0.00294 -> 0.294
- link act7Seg2helper_shape: mass 2.94e-06 -> 0.000294
- link act7Seg3: mass 0.00294 -> 0.294
- link act7Seg3helper_shape: mass 2.94e-06 -> 0.000294
- link act7Seg4: mass 0.00294 -> 0.294
- link act7Seg4helper_shape: mass 2.94e-06 -> 0.000294
- link act7Seg5: mass 0.00294 -> 0.294
- link act7Seg5helper_shape: mass 2.94e-06 -> 0.000294
- link act8Seg0: mass 0.00294 -> 0.294
- link act8Seg1: mass 0.00294 -> 0.294
- link act8Seg1helper_shape: mass 2.94e-06 -> 0.000294
- link act8Seg2: mass 0.00294 -> 0.294
- link act8Seg2helper_shape: mass 2.94e-06 -> 0.000294
- link act8Seg3: mass 0.00294 -> 0.294
- link act8Seg3helper_shape: mass 2.94e-06 -> 0.000294
- link act8Seg4: mass 0.00294 -> 0.294
- link act8Seg4helper_shape: mass 2.94e-06 -> 0.000294
- link act8Seg5: mass 0.00294 -> 0.294
- link act8Seg5helper_shape: mass 2.94e-06 -> 0.000294
- link act9Seg0: mass 0.00294 -> 0.294
- link act9Seg1: mass 0.00294 -> 0.294
- link act9Seg1helper_shape: mass 2.94e-06 -> 0.000294
- link act9Seg2: mass 0.00294 -> 0.294
- link act9Seg2helper_shape: mass 2.94e-06 -> 0.000294
- link act9Seg3: mass 0.00294 -> 0.294
- link act9Seg3helper_shape: mass 2.94e-06 -> 0.000294
- link act9Seg4: mass 0.00294 -> 0.294
- link act9Seg4helper_shape: mass 2.94e-06 -> 0.000294
- link act9Seg5: mass 0.00294 -> 0.294
- link act9Seg5helper_shape: mass 2.94e-06 -> 0.000294
